Commit message: added urdf with zeppelin

File: dev_ws/src/sam_bot_description/src/description/sam_bot_description.urdf (robot description, URDF)
Before this commit: robot sam_bot, 7 links, 6 joints
Links:
- removed link camera_depth_frame
- removed link camera_link
- removed link front_caster
- added link carbon_rod; collision cylinder length=${carbon_rod_length} radius=0.007; visual cylinder length=${carbon_rod_length} radius=0.007
- added link computer_link; visual box size=0.15 0.07 ${haul_over_ground*0.6}
- added link haul; collision box size=${haul_length} ${haul_width} ${haul_width}; visual cylinder length=${haul_length-haul_width} radius=${haul_width/2}
- added link wheel_left; collision cylinder length=${wheel_width} radius=${wheel_radius}; visual cylinder length=${wheel_width} radius=${wheel_radius}
- added link wheel_right; collision cylinder length=${wheel_width} radius=${wheel_radius}; visual cylinder length=${wheel_width} radius=${wheel_radius}
- link base_link: geometry 
- link imu_link: geometry 
- link lidar_link: mass 0.125 -> None; geometry visual cylinder length=0.05 radius=0.05
Joints:
- removed joint camera_depth_joint
- removed joint camera_joint
- removed joint caster_joint
- added joint carbon_bar: type fixed, parent base_link, child carbon_rod, origin xyz=0.0 0.0 0 rpy=0 0 0
- added joint computer_joint: type fixed, parent base_link, child computer_link, origin xyz=0 0 ${-haul_over_ground*0.3} rpy=0 0 0
- added joint haul_joint: type fixed, parent base_link, child haul, origin xyz=0.0 0.0 ${haul_width/2} rpy=0 0 0
- added joint wheel_left_joint: type fixed, parent base_link, child wheel_left, origin xyz=0 ${carbon_rod_length/2} 0 rpy=0 0 0, axis 0 1 0
- added joint wheel_right_joint: type fixed, parent base_link, child wheel_right, origin xyz=0 ${-carbon_rod_length/2} 0 rpy=0 0 0, axis 0 1 0
- joint base_joint: origin xyz=0.0 0.0 ${-(wheel_radius+wheel_zoff)} rpy=0 0 0 -> xyz=0.0 0.0 ${-haul_over_ground} rpy=0 0 0
- joint imu_joint: origin xyz=0 0 0.01 -> xyz=0 0 0
- joint lidar_joint: origin xyz=0 0 0.12 rpy=0 0 0 -> xyz=0 0 ${-haul_over_ground+0.05/2} rpy=0 0 0

Commit message: remove unneeded parts

File: dev_ws/src/sam_bot_description/src/description/sam_bot_description.urdf (robot description, URDF)
Before this commit: robot sam_bot, 9 links, 8 joints
Links:
- removed link computer_link
Joints:
- removed joint computer_joint

Commit message: did shit

File: dev_ws/src/sam_bot_description/src/description/sam_bot_description.urdf (robot description, URDF)
Before this commit: robot sam_bot, 8 links, 7 joints
Links:
- added link cam_link
Joints:
- added joint cam_link: type fixed, parent base_link, child cam_link, origin xyz=0 0 0 rpy=${pi/-2} 0 ${pi/-2}
